File: CHore/CHore.kicad_pcb (KiCad board)
At the start: 2 copper layers, 214.8 x 117.2 mm, 76 parts, among them J1 Conn_01x02_Pin, J2 USB_C_Receptacle_USB2.0, J3 Conn_01x02_Pin, SW1 SW_PUSH, SW10 SW_PUSH, SW11 SW_PUSH, SW12 SW_PUSH, SW13 SW_PUSH, SW14 SW_PUSH, SW15 SW_PUSH, SW16 SW_PUSH, SW17 SW_PUSH, SW18 SW_PUSH, SW19 SW_PUSH, SW2 SW_PUSH, SW20 SW_PUSH, SW21 SW_PUSH, SW22 SW_PUSH, SW23 SW_PUSH, SW24 SW_PUSH, SW25 SW_PUSH, SW26 SW_PUSH, SW27 SW_PUSH, SW28 SW_PUSH, SW29 SW_PUSH, SW3 SW_PUSH, SW30 SW_PUSH, SW4 SW_PUSH, SW5 SW_PUSH, SW6 SW_PUSH, SW7 SW_PUSH, SW8 SW_PUSH, SW9 SW_PUSH, U1 CH552G

Commit message: Fixed hardware to prevent ghosting.
Parts:
- removed R5, R6, R7, R8, R9: 10k, PCM_Resistor_SMD_AKL:R_0603_1608Metric
- added D31: 1N4148W, Diode_SMD:D_SOD-123, B.Cu at (76.0, 53.4)
- added D32: 1N4148W, Diode_SMD:D_SOD-123, B.Cu at (93.6, 75.0)
- added D33: 1N4148W, Diode_SMD:D_SOD-123, B.Cu at (139.8, 98.2)
- added D34: 1N4148W, Diode_SMD:D_SOD-123, B.Cu at (182.2, 69.2)
- added D35: 1N4148W, Diode_SMD:D_SOD-123, B.Cu at (222.3, 54.7)
Connections:
- SW1 pad 1: /COL0 -> Net-(D31-K)
- SW11 pad 1: /COL0 -> Net-(D31-K)
- SW13 pad 1: /COL1 -> Net-(D32-K)
- SW15 pad 1: /COL2 -> Net-(D33-K)
- SW17 pad 1: /COL3 -> Net-(D34-K)
- SW19 pad 1: /COL4 -> Net-(D35-K)
- SW22 pad 1: /COL1 -> Net-(D32-K)
- SW24 pad 1: /COL3 -> Net-(D34-K)
- SW26 pad 1: /COL4 -> Net-(D35-K)
- SW28 pad 1: /COL2 -> Net-(D33-K)
- SW3 pad 1: /COL1 -> Net-(D32-K)
- SW30 pad 1: /COL3 -> Net-(D34-K)
- SW5 pad 1: /COL2 -> Net-(D33-K)
- SW7 pad 1: /COL3 -> Net-(D34-K)
- SW9 pad 1: /COL4 -> Net-(D35-K)
Routing:
- net /COL2: track 230.4 -> 100.9 mm, vias 3 -> 2
- net Net-(D34-K): track 0.00 -> 99.3 mm, vias 0 -> 3
- net Net-(D33-K): track 0.00 -> 95.7 mm, vias 0 -> 4
- net /COL3: track 189.0 -> 115.9 mm, vias 6 -> 4
- net /COL1: track 198.4 -> 145.1 mm, vias 7 -> 5
- net Net-(D32-K): track 0.00 -> 52.4 mm, vias 0 -> 3
- net Net-(D35-K): track 0.00 -> 52.3 mm, vias 0 -> 3
- net /3V3: track 73.3 -> 26.8 mm, vias 13 -> 4
- net Net-(D31-K): track 0.00 -> 43.8 mm
- net /COL0: track 174.9 -> 140.8 mm
- net /COL4: track 176.4 -> 146.9 mm, vias 5 -> 3
