File: CHore/CHore.kicad_sch (KiCad schematic)
At the start: 76 parts, among them J1 Conn_01x02_Pin, J2 USB_C_Receptacle_USB2.0, J3 Conn_01x02_Pin, SW1 SW_PUSH, SW10 SW_PUSH, SW11 SW_PUSH, SW12 SW_PUSH, SW13 SW_PUSH, SW14 SW_PUSH, SW15 SW_PUSH, SW16 SW_PUSH, SW17 SW_PUSH, SW18 SW_PUSH, SW19 SW_PUSH, SW2 SW_PUSH, SW20 SW_PUSH, SW21 SW_PUSH, SW22 SW_PUSH, SW23 SW_PUSH, SW24 SW_PUSH, SW25 SW_PUSH, SW26 SW_PUSH, SW27 SW_PUSH, SW28 SW_PUSH, SW29 SW_PUSH, SW3 SW_PUSH, SW30 SW_PUSH, SW4 SW_PUSH, SW5 SW_PUSH, SW6 SW_PUSH, SW7 SW_PUSH, SW8 SW_PUSH, SW9 SW_PUSH, U1 CH552G

Commit message: Fixed hardware to prevent ghosting.
Parts:
- removed R5, R6, R7, R8, R9: 10k, PCM_Resistor_SMD_AKL:R_0603_1608Metric, symbol Device:R
- added D31, D32, D33, D34, D35: 1N4148W, Diode_SMD:D_SOD-123, symbol Diode:1N4148W
Connections:
- net COL0: now also D31.2 (A); no longer SW1.1, SW11.1
- net COL1: now also D32.2 (A); no longer SW13.1, SW22.1, SW3.1
- net COL2: now also D33.2 (A); no longer SW15.1, SW28.1, SW5.1
- net COL3: now also D34.2 (A); no longer SW17.1, SW24.1, SW30.1, SW7.1
- net COL4: now also D35.2 (A); no longer SW19.1, SW26.1, SW9.1
- new net: D33.1 (K), SW15.1, SW28.1, SW5.1
- new net: D31.1 (K), SW1.1, SW11.1
- new net: D32.1 (K), SW13.1, SW22.1, SW3.1
- new net: D34.1 (K), SW17.1, SW24.1, SW30.1, SW7.1
- new net: D35.1 (K), SW19.1, SW26.1, SW9.1
